File: TractiveSystemPCBv2/RacingTeam.sch (KiCad schematic (older format))
At the start: 84 parts, among them J1 BusIn, J11 ShutdownIn, J2 Bypass Pin, J3 BypassPin, J4 BypassPin, J5 BypassPin, J6 PC Relay, J7 AIROut, J8 Discharge Relay Out, J9 Molex, Q1 TP0610T, Q2 2N7002, Q3 2N7002, Q4 TP0610T, Q5 2N7002, Q6 TP0610T, Q7 2N7002, Q8 TP0610T, Q9 TP0610T, U1 LM311, U2 LM311, U3 4N35, U4 MC78M12ABDTRKG, U6 NE555D

Commit message: Update GRC22Symbols.dcm, GRC22Symbols.lib, and 3 more files...
Parts:
- added R?: 1.2kΩ, GRC22Footprints:R_0603_1608Metric_Pad0.98x0.95mm_HandSolder, symbol GRC22Symbols:R
- added R?: 0Ω, GRC22Footprints:R_0805_2012Metric_Pad1.20x1.40mm_HandSolder, symbol GRC22Symbols:R
- added U?: 4N35, GRC22Footprints:OPTO_4N35SM, symbol GRC22Symbols:4N35SM
Connections:
- net +12V: now also PS1.6 (+VOUT), U?.1
- net +BATT: now also PS1.2 (+VIN)
- net GLV+: now also U?.5
- net GLV-: now also PS1.1 (-VIN)
- net GND: now also PS1.7 (-VOUT)
- net PrechargeBus: no longer D1.1 (K)
- net PrechargeCompOUT: no longer Q1.1 (G), Q2.1 (G), R20.1, U1.7
- net at R21.1: now also R?.1
- net PrechargeTP+: no longer names the net of F6.2, J3.1 (Pin_1), R16.2, R35.1
- net PrechargeTP+: now also D1.1 (K)
- new net: R20.1, R?.1, U1.7
- new net: Q1.1 (G), Q2.1 (G), R?.2, U?.4
- new net: R?.2, U?.2
- no-connect marks 1 -> 2
Other:
- note added: "Reference Voltage\n"
- note added: "Tractive System Voltage Divider"
- moved on the sheet: C1, C2, D1, D3, D4, F5, F6, J2, J3, J6, J7, Q1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

Commit message: Update RacingTeam.kicad_pcb-bak, RacingTeam.xml, and 38 more files...
Parts:
- removed C2: 0.1uF, GRC22Footprints:C_0603_1608Metric_Pad1.08x0.95mm_HandSolder, symbol Device:C
- removed C4: 0.1uF, GRC22Footprints:C_0603_1608Metric_Pad1.08x0.95mm_HandSolder, symbol GRC22Symbols:C
- removed D5: Flyback, GRC22Footprints:D_0805_2012Metric_Castellated, symbol Device:D
- removed F2, F5: Fuse_Small, GRC22Footprints:FUSE_0154004.DRTL, symbol Device:Fuse_Small
- removed J11: ShutdownIn, GRC22Footprints:CUI_TBL001-500-02GY-2GY, symbol Connector:Screw_Terminal_01x02
- removed J9: Molex, GRC22Footprints:Molex, symbol GRC22Symbols:Conn_01x06
- removed Q9: TP0610T, GRC22Footprints:2N7002H6327XTSA2_v2, symbol GRC22Symbols:RSC002P03T316
- removed R1, R2, R3: 1.3kΩ, GRC22Footprints:R_0603_1608Metric_Pad0.98x0.95mm_HandSolder, symbol GRC22Symbols:R
- removed R10, R8, R9: 150kΩ, GRC22Footprints:R_0805_2012Metric_Pad1.20x1.40mm_HandSolder, symbol Device:R
- removed R11: 4kΩ, GRC22Footprints:R_0805_2012Metric_Pad1.20x1.40mm_HandSolder, symbol Device:R
- removed R21, R23, R25, R34, R36, R?: 0Ω, GRC22Footprints:R_0805_2012Metric_Pad1.20x1.40mm_HandSolder, symbol GRC22Symbols:R
- removed R37: 4kΩ, GRC22Footprints:R_0603_1608Metric_Pad0.98x0.95mm_HandSolder, symbol GRC22Symbols:R
- removed R4: 4.7kΩ, GRC22Footprints:R_0603_1608Metric_Pad0.98x0.95mm_HandSolder, symbol Device:R
- removed R5: 6.8kΩ, GRC22Footprints:R_0603_1608Metric_Pad0.98x0.95mm_HandSolder, symbol Device:R
- removed R7: 22kΩ, GRC22Footprints:R_0805_2012Metric_Pad1.20x1.40mm_HandSolder, symbol GRC22Symbols:R
- added C1, C2: 470nF, TractiveSystemLib:C_0603_1608Metric_Pad1.08x0.95mm_HandSolder, symbol TractiveSystemPCBv2:C
- added C12: 1μF, TractiveSystemLib:C_0603_1608Metric_Pad1.08x0.95mm_HandSolder, symbol TractiveSystemPCBv2:C
- added C3, C4: 22μF, TractiveSystemLib:CAPE830X690N, symbol TractiveSystemPCBv2:CP1
- added D5: Flyback, TractiveSystemLib:D_0805_2012Metric_Castellated, symbol TractiveSystemPCBv2:D
- added D7: D, TractiveSystemLib:D_0805_2012Metric_Castellated, symbol TractiveSystemPCBv2:D
- added J2: PowerInput, TractiveSystemLib:CUI_TBL001-500-02GY-2GY, symbol TractiveSystemPCBv2:Conn_01x02
- added J3: BrakePositionSensor, TractiveSystemLib:CUI_TBL001-500-02GY-2GY, symbol TractiveSystemPCBv2:Conn_01x02
- added J4: StartButton, TractiveSystemLib:CUI_TBL001-500-02GY-2GY, symbol TractiveSystemPCBv2:Conn_01x02
- added J5: Molex, TractiveSystemLib:878310819, symbol TractiveSystemPCBv2:Conn_01x08
- added Q10: FMMT494QTA, TractiveSystemLib:SOT91P240X110-3N, symbol TractiveSystemPCBv2:Q_NPN_BCE
- added Q11: RSC, TractiveSystemLib:BZT03C12-TR, symbol TractiveSystemPCBv2:Q_PMOS_GSD
- added Q8: RSC002, TractiveSystemLib:BZT03C12-TR, symbol TractiveSystemPCBv2:Q_PMOS_GSD
- added R1, R2: 200kΩ, TractiveSystemLib:R_0805_2012Metric_Pad1.20x1.40mm_HandSolder, symbol TractiveSystemPCBv2:R
- added R10, R9: 1kΩ, TractiveSystemLib:R_0603_1608Metric_Pad0.98x0.95mm_HandSolder, symbol TractiveSystemPCBv2:R
- added R22, R28: 10kΩ, TractiveSystemLib:R_0603_1608Metric_Pad0.98x0.95mm_HandSolder, symbol TractiveSystemPCBv2:R
- added R3: 25kΩ, TractiveSystemLib:R_0805_2012Metric_Pad1.20x1.40mm_HandSolder, symbol TractiveSystemPCBv2:R
- added R30: 47kΩ, TractiveSystemLib:R_0603_1608Metric_Pad0.98x0.95mm_HandSolder, symbol TractiveSystemPCBv2:R
- added R31: 4.7kΩ, TractiveSystemLib:R_0603_1608Metric_Pad0.98x0.95mm_HandSolder, symbol TractiveSystemPCBv2:R
- added RV1, RV2: 10kΩ, TractiveSystemLib:PT01-D120K2-B103, symbol TractiveSystemPCBv2:R_POT
- added U1, U2: LM2941LD, TractiveSystemLib:DFN400X400X80-9N, symbol TractiveSystemPCBv2:LM2941LD
- C10: renamed from C9; footprint GRC22Footprints:C_0603_1608Metric_Pad1.08x0.95mm_HandSolder -> TractiveSystemLib:C_0603_1608Metric_Pad1.08x0.95mm_HandSolder; symbol GRC22Symbols:C -> TractiveSystemPCBv2:C
- C11: renamed from C10; footprint GRC22Footprints:C_0603_1608Metric_Pad1.08x0.95mm_HandSolder -> TractiveSystemLib:C_0603_1608Metric_Pad1.08x0.95mm_HandSolder; symbol GRC22Symbols:C -> TractiveSystemPCBv2:C
- C5: renamed from C1; footprint GRC22Footprints:C_0603_1608Metric_Pad1.08x0.95mm_HandSolder -> TractiveSystemLib:C_0603_1608Metric_Pad1.08x0.95mm_HandSolder; symbol GRC22Symbols:C -> TractiveSystemPCBv2:C
- C6: renamed from C3; footprint GRC22Footprints:C_0603_1608Metric_Pad1.08x0.95mm_HandSolder -> TractiveSystemLib:C_0603_1608Metric_Pad1.08x0.95mm_HandSolder; symbol GRC22Symbols:C -> TractiveSystemPCBv2:C
- C7: renamed from C5; footprint GRC22Footprints:C_0603_1608Metric_Pad1.08x0.95mm_HandSolder -> TractiveSystemLib:C_0603_1608Metric_Pad1.08x0.95mm_HandSolder; symbol GRC22Symbols:C -> TractiveSystemPCBv2:C
- C8: renamed from C6; footprint GRC22Footprints:C_0603_1608Metric_Pad1.08x0.95mm_HandSolder -> TractiveSystemLib:C_0603_1608Metric_Pad1.08x0.95mm_HandSolder; symbol GRC22Symbols:C -> TractiveSystemPCBv2:C
- C9: renamed from C8; footprint GRC22Footprints:C_0603_1608Metric_Pad1.08x0.95mm_HandSolder -> TractiveSystemLib:C_0603_1608Metric_Pad1.08x0.95mm_HandSolder; symbol GRC22Symbols:C -> TractiveSystemPCBv2:C
- D1: renamed from D2; footprint GRC22Footprints:SOD57-10 -> TractiveSystemLib:SOD57-10; symbol GRC22Symbols:D -> TractiveSystemPCBv2:D_Zener
- D2: renamed from D1; footprint GRC22Footprints:SOD57-10 -> TractiveSystemLib:SOD57-10; symbol GRC22Symbols:D -> TractiveSystemPCBv2:D_Zener
- D3: renamed from D6; footprint GRC22Footprints:D_0603_1608Metric_Castellated -> TractiveSystemLib:D_0805_2012Metric_Castellated; symbol GRC22Symbols:D -> TractiveSystemPCBv2:LED
- D4: footprint GRC22Footprints:D_0805_2012Metric_Castellated -> TractiveSystemLib:D_0805_2012Metric_Castellated; symbol Device:D -> TractiveSystemPCBv2:D
- D6: renamed from D3; footprint GRC22Footprints:D_0805_2012Metric_Castellated -> TractiveSystemLib:D_0805_2012Metric_Castellated; symbol Device:D -> TractiveSystemPCBv2:D
- D8: footprint GRC22Footprints:D_0603_1608Metric_Castellated -> TractiveSystemLib:D_0805_2012Metric_Castellated; symbol GRC22Symbols:D -> TractiveSystemPCBv2:LED
- F1: footprint GRC22Footprints:FUSE_0154004.DRTL -> TractiveSystemLib:FUSE_0154004.DRTL; symbol Device:Fuse_Small -> TractiveSystemPCBv2:Fuse
- F2: renamed from F6; footprint GRC22Footprints:FUSE_0154004.DRTL -> TractiveSystemLib:FUSE_0154004.DRTL; symbol Device:Fuse_Small -> TractiveSystemPCBv2:Fuse
- J1: footprint GRC22Footprints:TE_8PCV-02-006 -> TractiveSystemLib:TE_8PCV-02-006; symbol Connector_Generic:Conn_01x02 -> TractiveSystemPCBv2:Conn_01x02
- J10: renamed from J3; footprint GRC22Footprints:PinHeader_1x01_P2.54mm_Vertical -> TractiveSystemLib:PinHeader_1x01_P2.54mm_Vertical; symbol Connector_Generic:Conn_01x01 -> TractiveSystemPCBv2:Conn_01x01
- J11: renamed from J7; value AIROut -> AIR Out; footprint GRC22Footprints:CUI_TBL001-500-02GY-2GY -> TractiveSystemLib:CUI_TBL001-500-02GY-2GY; symbol Connector:Screw_Terminal_01x02 -> TractiveSystemPCBv2:Conn_01x02
- J12: renamed from J8; value Discharge Relay Out -> DischargeRelay; footprint GRC22Footprints:CUI_TBL001-500-02GY-2GY -> TractiveSystemLib:CUI_TBL001-500-02GY-2GY; symbol Connector:Screw_Terminal_01x02 -> TractiveSystemPCBv2:Conn_01x02
- J6: renamed from J4; footprint GRC22Footprints:PinHeader_1x01_P2.54mm_Vertical -> TractiveSystemLib:PinHeader_1x01_P2.54mm_Vertical; symbol Connector_Generic:Conn_01x01 -> TractiveSystemPCBv2:Conn_01x01
- J7: renamed from J2; value Bypass Pin -> TSW-101-23-S-S; footprint GRC22Footprints:PinHeader_1x01_P2.54mm_Vertical -> TractiveSystemLib:PinHeader_1x01_P2.54mm_Vertical; symbol Connector_Generic:Conn_01x01 -> TractiveSystemPCBv2:Conn_01x01
- J8: renamed from J5; footprint GRC22Footprints:PinHeader_1x01_P2.54mm_Vertical -> TractiveSystemLib:PinHeader_1x01_P2.54mm_Vertical; symbol Connector_Generic:Conn_01x01 -> TractiveSystemPCBv2:Conn_01x01
- J9: renamed from J6; value PC Relay -> PC Out; footprint GRC22Footprints:CUI_TBL001-500-02GY-2GY -> TractiveSystemLib:CUI_TBL001-500-02GY-2GY; symbol Connector:Screw_Terminal_01x02 -> TractiveSystemPCBv2:Conn_01x02
- JP1, JP2: footprint GRC22Footprints:PinHeader_1x02_P2.54mm_Vertical -> TractiveSystemLib:PinHeader_1x02_P2.54mm_Vertical; symbol GRC22Symbols:Jumper -> TractiveSystemPCBv2:Jumper
- PS1: footprint GRC22Footprints:CONV_SPBW06F-12 -> TractiveSystemLib:CONV_SPBW06F-12; symbol GRC22Symbols:SPBW06F-12 -> TractiveSystemPCBv2:SPBW06F-12
- Q1: renamed from Q5; footprint GRC22Footprints:2N7002H6327XTSA2 -> TractiveSystemLib:2N7002H6327XTSA2; symbol GRC22Symbols:2N7002 -> TractiveSystemPCBv2:Q_NMOS_GSD
- Q2: renamed from Q3; footprint GRC22Footprints:2N7002H6327XTSA2 -> TractiveSystemLib:2N7002H6327XTSA2; symbol GRC22Symbols:2N7002 -> TractiveSystemPCBv2:Q_NMOS_GSD
- Q3: renamed from Q2; footprint GRC22Footprints:2N7002H6327XTSA2 -> TractiveSystemLib:2N7002H6327XTSA2; symbol GRC22Symbols:2N7002 -> TractiveSystemPCBv2:Q_NMOS_GSD
- Q4: renamed from Q6; value TP0610T -> RSC002; footprint GRC22Footprints:2N7002H6327XTSA2_v2 -> TractiveSystemLib:BZT03C12-TR; symbol GRC22Symbols:RSC002P03T316 -> TractiveSystemPCBv2:Q_PMOS_GSD
- Q5: renamed from Q4; value TP0610T -> RSC002; footprint GRC22Footprints:2N7002H6327XTSA2_v2 -> TractiveSystemLib:BZT03C12-TR; symbol GRC22Symbols:RSC002P03T316 -> TractiveSystemPCBv2:Q_PMOS_GSD
- Q6: renamed from Q1; value TP0610T -> RSC002; footprint GRC22Footprints:2N7002H6327XTSA2_v2 -> TractiveSystemLib:BZT03C12-TR; symbol GRC22Symbols:RSC002P03T316 -> TractiveSystemPCBv2:Q_PMOS_GSD
- Q7: footprint GRC22Footprints:2N7002H6327XTSA2 -> TractiveSystemLib:2N7002H6327XTSA2; symbol GRC22Symbols:2N7002 -> TractiveSystemPCBv2:Q_NMOS_GSD
- Q9: renamed from Q8; value TP0610T -> RSC002; footprint GRC22Footprints:2N7002H6327XTSA2_v2 -> TractiveSystemLib:BZT03C12-TR; symbol GRC22Symbols:RSC002P03T316 -> TractiveSystemPCBv2:Q_PMOS_GSD
- R11: renamed from R33; footprint GRC22Footprints:R_0805_2012Metric_Pad1.20x1.40mm_HandSolder -> TractiveSystemLib:R_0603_1608Metric_Pad0.98x0.95mm_HandSolder; symbol GRC22Symbols:R -> TractiveSystemPCBv2:R
- R12: renamed from R35; footprint GRC22Footprints:R_0805_2012Metric_Pad1.20x1.40mm_HandSolder -> TractiveSystemLib:R_0603_1608Metric_Pad0.98x0.95mm_HandSolder; symbol GRC22Symbols:R -> TractiveSystemPCBv2:R
- R14: renamed from R18; footprint GRC22Footprints:R_0603_1608Metric_Pad0.98x0.95mm_HandSolder -> TractiveSystemLib:R_0603_1608Metric_Pad0.98x0.95mm_HandSolder; symbol GRC22Symbols:R -> TractiveSystemPCBv2:R
- R15: renamed from R19; footprint GRC22Footprints:R_0603_1608Metric_Pad0.98x0.95mm_HandSolder -> TractiveSystemLib:R_0603_1608Metric_Pad0.98x0.95mm_HandSolder; symbol GRC22Symbols:R -> TractiveSystemPCBv2:R
- R16: renamed from R17; footprint GRC22Footprints:R_0603_1608Metric_Pad0.98x0.95mm_HandSolder -> TractiveSystemLib:R_0603_1608Metric_Pad0.98x0.95mm_HandSolder; symbol GRC22Symbols:R -> TractiveSystemPCBv2:R
- R17: renamed from R16; footprint GRC22Footprints:R_0603_1608Metric_Pad0.98x0.95mm_HandSolder -> TractiveSystemLib:R_0603_1608Metric_Pad0.98x0.95mm_HandSolder; symbol GRC22Symbols:R -> TractiveSystemPCBv2:R
- R18: renamed from R22; footprint GRC22Footprints:R_0603_1608Metric_Pad0.98x0.95mm_HandSolder -> TractiveSystemLib:R_0603_1608Metric_Pad0.98x0.95mm_HandSolder; symbol GRC22Symbols:R -> TractiveSystemPCBv2:R
- R19: renamed from R20; footprint GRC22Footprints:R_0603_1608Metric_Pad0.98x0.95mm_HandSolder -> TractiveSystemLib:R_0603_1608Metric_Pad0.98x0.95mm_HandSolder; symbol GRC22Symbols:R -> TractiveSystemPCBv2:R
- R20: renamed from R?; footprint GRC22Footprints:R_0603_1608Metric_Pad0.98x0.95mm_HandSolder -> TractiveSystemLib:R_0603_1608Metric_Pad0.98x0.95mm_HandSolder; symbol GRC22Symbols:R -> TractiveSystemPCBv2:R
- R21: renamed from R24; footprint GRC22Footprints:R_0603_1608Metric_Pad0.98x0.95mm_HandSolder -> TractiveSystemLib:R_0603_1608Metric_Pad0.98x0.95mm_HandSolder; symbol GRC22Symbols:R -> TractiveSystemPCBv2:R
- R23: renamed from R26; footprint GRC22Footprints:R_0603_1608Metric_Pad0.98x0.95mm_HandSolder -> TractiveSystemLib:R_0603_1608Metric_Pad0.98x0.95mm_HandSolder; symbol GRC22Symbols:R -> TractiveSystemPCBv2:R
- R24: renamed from R27; footprint GRC22Footprints:R_0603_1608Metric_Pad0.98x0.95mm_HandSolder -> TractiveSystemLib:R_0603_1608Metric_Pad0.98x0.95mm_HandSolder; symbol GRC22Symbols:R -> TractiveSystemPCBv2:R
- R25: renamed from R28; footprint GRC22Footprints:R_0603_1608Metric_Pad0.98x0.95mm_HandSolder -> TractiveSystemLib:R_0603_1608Metric_Pad0.98x0.95mm_HandSolder; symbol GRC22Symbols:R -> TractiveSystemPCBv2:R
- R26: renamed from R29; footprint GRC22Footprints:R_0603_1608Metric_Pad0.98x0.95mm_HandSolder -> TractiveSystemLib:R_0603_1608Metric_Pad0.98x0.95mm_HandSolder; symbol GRC22Symbols:R -> TractiveSystemPCBv2:R
- R27: renamed from R30; footprint GRC22Footprints:R_0603_1608Metric_Pad0.98x0.95mm_HandSolder -> TractiveSystemLib:R_0603_1608Metric_Pad0.98x0.95mm_HandSolder; symbol GRC22Symbols:R -> TractiveSystemPCBv2:R
- R29: renamed from R31; footprint GRC22Footprints:R_0603_1608Metric_Pad0.98x0.95mm_HandSolder -> TractiveSystemLib:R_0603_1608Metric_Pad0.98x0.95mm_HandSolder; symbol GRC22Symbols:R -> TractiveSystemPCBv2:R
- R32: footprint GRC22Footprints:R_0603_1608Metric_Pad0.98x0.95mm_HandSolder -> TractiveSystemLib:R_0603_1608Metric_Pad0.98x0.95mm_HandSolder; symbol GRC22Symbols:R -> TractiveSystemPCBv2:R
- R4: renamed from R6; value 249kΩ -> 500kΩ; footprint GRC22Footprints:R_0805_2012Metric_Pad1.20x1.40mm_HandSolder -> TractiveSystemLib:R_0805_2012Metric_Pad1.20x1.40mm_HandSolder; symbol GRC22Symbols:R -> TractiveSystemPCBv2:R
- R5: renamed from R12; value 249kΩ -> 500kΩ; footprint GRC22Footprints:R_0805_2012Metric_Pad1.20x1.40mm_HandSolder -> TractiveSystemLib:R_0805_2012Metric_Pad1.20x1.40mm_HandSolder; symbol GRC22Symbols:R -> TractiveSystemPCBv2:R
- R6: renamed from R13; value 249kΩ -> 150kΩ; footprint GRC22Footprints:R_0805_2012Metric_Pad1.20x1.40mm_HandSolder -> TractiveSystemLib:R_0805_2012Metric_Pad1.20x1.40mm_HandSolder; symbol GRC22Symbols:R -> TractiveSystemPCBv2:R
- R7: renamed from R14; value 249kΩ -> 150kΩ; footprint GRC22Footprints:R_0805_2012Metric_Pad1.20x1.40mm_HandSolder -> TractiveSystemLib:R_0805_2012Metric_Pad1.20x1.40mm_HandSolder; symbol GRC22Symbols:R -> TractiveSystemPCBv2:R
- R8: renamed from R15; value 49kΩ -> 25kΩ; footprint GRC22Footprints:R_0805_2012Metric_Pad1.20x1.40mm_HandSolder -> TractiveSystemLib:R_0805_2012Metric_Pad1.20x1.40mm_HandSolder; symbol GRC22Symbols:R -> TractiveSystemPCBv2:R
- U3: renamed from U1; footprint GRC22Footprints:LM311PW -> TractiveSystemLib:LM311PW; symbol GRC22Symbols:LM311 -> TractiveSystemPCBv2:LM311
- U4: renamed from U2; footprint GRC22Footprints:LM311PW -> TractiveSystemLib:LM311PW; symbol GRC22Symbols:LM311 -> TractiveSystemPCBv2:LM311
- U5: renamed from U?; footprint GRC22Footprints:OPTO_4N35SM -> TractiveSystemLib:OPTO_4N35SM; symbol GRC22Symbols:4N35SM -> TractiveSystemPCBv2:4N35SM
- U6: renamed from U3; footprint GRC22Footprints:OPTO_4N35SM -> TractiveSystemLib:OPTO_4N35SM; symbol GRC22Symbols:4N35SM -> TractiveSystemPCBv2:4N35SM
- U7: renamed from U6; footprint GRC22Footprints:NE555PSRE4 -> TractiveSystemLib:NE555PSRE4; symbol GRC22Symbols:NE555D -> TractiveSystemPCBv2:NE555D
- U8: renamed from U4; footprint GRC22Footprints:TO229P990X238-4N -> TractiveSystemLib:TO229P990X238-4N; symbol GRC22Symbols:MC78M12ABDTRKG -> TractiveSystemPCBv2:MC78M12ABDTRKG
Connections:
- net labels added: AIR+, BusOutPrecharge, Common, Discharge, Precharge-, PrechargeOPTO, PrechargeRef, RTDLatch, RTDOutput, RTDReady
- net labels removed: AIRON, DischargeIn, DischargeOut, Enable, PreChargeON, PrechargeBus, PrechargeRef2, PrechargeRelayOut, PrechargeTP-, Shutdown, TSALREFOut
- wire segments 204 -> 233
- no-connect marks 2 -> 5
Other:
- note added: "AIR\n\n\n"
- note added: "BoardInputs\n\n\n"
- note added: "BoardOutputs\n"
- note added: "Latch Activation\n"
- note added: "PCR\n\n\n\n"
- note added: "Precharge\nTrigger Voltage = 525V\nVoltage Division Ratio = 0.9857\n525V- 525(0.9857) = 7.5V"
- note added: "Ready To Drive\n\n\n\n"
- note added: "RelayOutputs\n\n"
- note added: "TSAL\nTrigger Voltage = 60V\nVoltage Division Ratio = 0.8857\n60V- 60(0.8857) = 6.86V"
- note added: "Trim Pot to 5.4k"
- note added: "Trim Pot to 5.9k"
- note removed: "ConnectorsIn\n\n"
- note removed: "ConnectorsOut\n\n\n"
- note removed: "Drain\nGate\nSource"
- note removed: "Power Enable\n\n\n"
- note removed: "Reference Voltage\n"
- note removed: "Schematic Notes\n\n\n"
- note removed: "The Enable Pin on the isolated HV GLV Regulator is controlled via the Shutdown Circuit, if the Shutdown Circuit is not active,\nno HV components will power on, but the GLV side will still remain on (From Battery to GLV regulator) to display a Green\nlight indicating safe voltages present inside the accumulator\n"
- note removed: "The SPBW06F-12 provides isloated 12V from the GLV to the HV side to power any components on the HV side as well as\nprovide the reference voltages for Voltage Divider Circuits\n"
- note removed: "Tractive System Voltage Divider"
- note removed: "Trigger Voltage = 60V\nVoltage Division Ratio = 0.93345\n60V- 60(0.93345) = 4V"
- moved on the sheet: C10, C11, C5, D2, D4, D6, F2, J1, J10, J7, J8, PS1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

Commit message: Update GRC Logo.jpg, GRCLogo.kicad_mod, and 21 more files...
Parts:
- removed C1, C2: 470nF, TractiveSystemLib:C_0603_1608Metric_Pad1.08x0.95mm_HandSolder, symbol TractiveSystemPCBv2:C
- removed C3, C4: 22μF, TractiveSystemLib:CAPE830X690N, symbol TractiveSystemPCBv2:CP1
- removed R10, R9: 1kΩ, TractiveSystemLib:R_0603_1608Metric_Pad0.98x0.95mm_HandSolder, symbol TractiveSystemPCBv2:R
- removed U1, U2: LM2941LD, TractiveSystemLib:DFN400X400X80-9N, symbol TractiveSystemPCBv2:LM2941LD
- J10: value BypassPin -> TSW-101-23-S-S
- renumbered C6 to C1, C5 to C2, C10 to C3, C11 to C4, C12 to C5, C9 to C6
Connections:
- wire segments 233 -> 192
- no-connect marks 5 -> 3
Other:
- note added: "Do not run AIR and relays through regulator"
- moved on the sheet: D5, J12, J2, J4, J6, RV2
