File: BSPD 2.0/bspd6.0_EDIT.kicad_sch (KiCad schematic)
At the start: 42 parts, among them J1 Brake Sensor Input, J2 Accumulator Sensor Input, J3 BSPD Sensor Output, Q1 RSC002, Q2 RSC002, Q3 RSC002, Q4 RSC002, Q5 RSC002, Q6 RSC002, Q7 RSC002, U1 LM311, U2 LM311, U3 LM311, U4 LM311, U5 ANDgate, U6 ANDgate, U7 MC78M12ABDTRKG, U8 LM311

Commit message: Update bspd6.0_EDIT.kicad_sch
Parts:
- removed U6: ANDgate, symbol bspd-cache:bspdlibrary_ANDgate
Other:
- moved on the sheet: J1, J2, J3, Q3, Q4, Q5, Q7, R11
